File: KiCad/USB-Hub V2.0.kicad_pcb (KiCad board)
At the start: 2 copper layers, 90 x 50 mm, 61 parts, among them IC1 XR22404, J1 USB_B_WE, J2 Conn_01x01, J3 Conn_01x01, J4 Conn_01x01, J5 Conn_01x01, J6 USB_A_shielded, J7 USB_A_shielded, J8 USB_A_shielded, J9 USB_A_shielded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

Commit message: Add files via upload
Parts:
- moved R4 190.3 mm to (101.8, 103.3)
- moved TP1 165.5 mm to (95.0, 111.6)
- moved R7 160.8 mm to (110.4, 102.0), turned to 180 degrees
- moved Q1 156.3 mm to (101.8, 110.6), turned to 270 degrees
- moved C1 154.9 mm to (101.8, 106.6)
- moved R6 152.6 mm to (134.4, 127.8)
- moved C2 149.7 mm to (108.5, 110.2), turned to 90 degrees
- moved R8 145.8 mm to (130.3, 105.3), turned to 270 degrees
- moved R5 142.6 mm to (112.0, 110.2), turned to 270 degrees
- moved F1 141.8 mm to (125.2, 111.6)
- moved Y1 135.0 mm to (146.6, 91.4), turned to 180 degrees
- moved C3 132.8 mm to (110.4, 105.3), turned to 180 degrees
- moved TP5 126.7 mm to (124.3, 102.4)
- moved D2 46.9 mm to (151.0, 109.5)
- moved D3 46.9 mm to (155.0, 109.5)
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Connections:
- FL1 pad 1: /USB_D_2- -> /USB_D_2+
- FL1 pad 2: USB_D_3- -> USB_D_3+
- FL1 pad 3: USB_D_3+ -> USB_D_3-
- FL1 pad 4: /USB_D_2+ -> /USB_D_2-
- IC1 pad 12: (no net) -> Net-(IC1-Pad12)
- IC1 pad 13: (no net) -> Net-(IC1-Pad13)
- IC1 pad 25: (no net) -> Net-(IC1-Pad25)
- IC1 pad 27: (no net) -> Net-(IC1-Pad27)
- IC1 pad 28: (no net) -> Net-(IC1-Pad28)
- J2 pad 1: (no net) -> Net-(J2-Pad1)
- J3 pad 1: (no net) -> Net-(J3-Pad1)
- J4 pad 1: (no net) -> Net-(J4-Pad1)
- J5 pad 1: (no net) -> Net-(J5-Pad1)
- U1 pad 1: /USB_D_2+ -> /USB_D_1-
- U1 pad 3: /USB_D_2- -> /USB_D_1+
- U1 pad 4: /USB_D_1- -> /USB_D_2+
- U1 pad 6: /USB_D_1+ -> /USB_D_2-
Routing:
- net VCC_5V: track 0.00 -> 45.8 mm, vias 0 -> 2
- net VBUS_SENSE: track 0.00 -> 35.9 mm
- net LED_CTL: track 0.00 -> 35.0 mm
- net LED2: track 0.00 -> 27.2 mm
- net GND: track 0.00 -> 23.8 mm, vias 0 -> 6
- net OSC1_in: track 0.00 -> 22.6 mm
- net LED1: track 0.00 -> 19.9 mm
- net USB_D_3+: track 0.00 -> 15.3 mm
- net Net-(IC1-Pad17): track 0.00 -> 15.1 mm
- net USB_D_3-: track 0.00 -> 14.8 mm
- net /USB_D_1+: track 0.00 -> 14.0 mm
- net VBUS_UP_P: track 0.00 -> 14.0 mm
- net /USB_D_1-: track 0.00 -> 11.4 mm
- net /USB_D_2+: track 0.00 -> 9.94 mm
- net /USB_D_2-: track 0.00 -> 9.94 mm
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- added copper zone on B.Cu, net GND
Other:
- net class 5V added: clearance 0.2, trace_width 0.75, via_dia 0.6, via_drill 0.4
- net class GND added: clearance 0.2, trace_width 0.75, via_dia 0.6, via_drill 0.4
- net class IC added: clearance 0.2, trace_width 0.35, via_dia 0.25, via_drill 0.2
- net class LED added: clearance 0.2, trace_width 0.75, via_dia 0.6, via_drill 0.2
- net class USB added: clearance 0.2, trace_width 0.15, via_dia 0.4, via_drill 0.2
- rule trace_min: 0.2 -> 0.1
- rule via_min_drill: 0.3 -> 0.2
- rule via_min_size: 0.4 -> 0.25
- board text added: "Active"
- board text added: "P1"
- board text added: "P2"
- board text added: "P3"
- board text added: "P4"

Commit message: no message
Connections:
- IC1 pad 12: Net-(IC1-Pad12) -> (no net)
- IC1 pad 13: Net-(IC1-Pad13) -> (no net)
- IC1 pad 25: Net-(IC1-Pad25) -> (no net)
- IC1 pad 27: Net-(IC1-Pad27) -> (no net)
- IC1 pad 28: Net-(IC1-Pad28) -> (no net)
- J2 pad 1: Net-(J2-Pad1) -> (no net)
- J3 pad 1: Net-(J3-Pad1) -> (no net)
- J4 pad 1: Net-(J4-Pad1) -> (no net)
- J5 pad 1: Net-(J5-Pad1) -> (no net)

Commit message: no message
Parts:
- added Txt2: OSHW, Symbols:OSHW-Logo2_7.3x6mm_SilkScreen, F.Cu at (169.7, 84.5)
- C10, C11, C12, C13, C6, C7, C8, C9, L1, L2, L3, L4: moved to B.Cu
- moved Txt1 185.0 mm to (170.3, 98.0), turned to 90 degrees
- moved C5 183.2 mm to (119.7, 107.1), turned to 180 degrees
- moved C4 178.5 mm to (119.7, 109.3)
- moved FL2 163.4 mm to (150.4, 86.5)
- moved TP2 160.9 mm to (136.0, 108.5)
- moved FL3 158.1 mm to (144.1, 84.3)
- moved FL5 156.6 mm to (106.2, 92.6), turned to 180 degrees
- moved C11 155.6 mm to (137.6, 79.8), turned to 180 degrees
- moved L1 154.4 mm to (160.3, 81.1), turned to 90 degrees
- moved FL4 151.4 mm to (127.9, 87.7), turned to 180 degrees
- moved L4 144.5 mm to (107.4, 84.2)
- moved L3 142.7 mm to (123.4, 82.2)
- moved C10 142.5 mm to (165.1, 79.8)
- moved U3 142.5 mm to (147.5, 80.3), turned to 90 degrees
- moved TP4 141.5 mm to (144.4, 103.7)
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Connections:
- FL2 pad 1: /DM4_1+ -> /DM4_1-
- FL2 pad 2: /DM4_2+ -> /DM4_2-
- FL2 pad 3: /DM4_2- -> /DM4_2+
- FL2 pad 4: /DM4_1- -> /DM4_1+
- FL3 pad 1: /DM3_1+ -> /DM3_1-
- FL3 pad 2: /DM3_2+ -> /DM3_2-
- FL3 pad 3: /DM3_2- -> /DM3_2+
- FL3 pad 4: /DM3_1- -> /DM3_1+
- FL4 pad 1: /DM2_1+ -> /DM2_1-
- FL4 pad 2: /DM2_2+ -> /DM2_2-
- FL4 pad 3: /DM2_2- -> /DM2_2+
- FL4 pad 4: /DM2_1- -> /DM2_1+
- FL5 pad 1: /DM1_1+ -> /DM1_1-
- FL5 pad 2: /DM1_2+ -> /DM1_2-
- FL5 pad 3: /DM1_2- -> /DM1_2+
- FL5 pad 4: /DM1_1- -> /DM1_1+
- IC1 pad 12: (no net) -> Net-(IC1-Pad12)
- IC1 pad 13: (no net) -> Net-(IC1-Pad13)
- IC1 pad 25: (no net) -> Net-(IC1-Pad25)
- IC1 pad 27: (no net) -> Net-(IC1-Pad27)
- IC1 pad 28: (no net) -> Net-(IC1-Pad28)
- J2 pad 1: (no net) -> Net-(J2-Pad1)
- J3 pad 1: (no net) -> Net-(J3-Pad1)
- J4 pad 1: (no net) -> Net-(J4-Pad1)
- J5 pad 1: (no net) -> Net-(J5-Pad1)
- U2 pad 1: /DM4_2- -> /DM4_2+
- U2 pad 3: /DM4_2+ -> /DM4_2-
- U2 pad 4: /DM4_3+ -> /DM4_3-
- U2 pad 6: /DM4_3- -> /DM4_3+
- U3 pad 1: /DM3_2- -> /DM3_2+
- U3 pad 3: /DM3_2+ -> /DM3_2-
- U3 pad 4: /DM3_3+ -> /DM3_3-
- U3 pad 6: /DM3_3- -> /DM3_3+
- U4 pad 1: /DM2_2- -> /DM2_2+
- U4 pad 3: /DM2_2+ -> /DM2_2-
- U4 pad 4: /DM2_3+ -> /DM2_3-
- U4 pad 6: /DM2_3- -> /DM2_3+
- U5 pad 1: /DM1_2- -> /DM1_2+
- U5 pad 3: /DM1_2+ -> /DM1_2-
- U5 pad 4: /DM1_3+ -> /DM1_3-
- U5 pad 6: /DM1_3- -> /DM1_3+
Routing:
- net VCC_5V: track 45.8 -> 192.6 mm, vias 2 -> 6
- net GND: track 23.8 -> 101.4 mm, vias 6 -> 11
- net VCC33: track 0.00 -> 35.5 mm, vias 0 -> 2
- net /DM1_1-: track 0.00 -> 31.0 mm
- net /DM1_1+: track 0.00 -> 30.7 mm
- net Net-(IC1-Pad19): track 0.00 -> 24.5 mm
- net OVC: track 0.00 -> 22.2 mm, vias 0 -> 2
- net /DM4_1+: track 0.00 -> 15.9 mm
- net Net-(IC1-Pad14): track 0.00 -> 15.8 mm
- net /DM4_1-: track 0.00 -> 15.4 mm
- net /DM3_1+: track 0.00 -> 13.9 mm
- net /DM3_2-: track 0.00 -> 13.5 mm
- net /DM4_2-: track 0.00 -> 13.4 mm
- net /DM3_1-: track 0.00 -> 13.4 mm
- net /DM4_2+: track 0.00 -> 12.9 mm
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