File: KiCad/USB-Hub V2.0.sch (KiCad schematic (older format))
At the start: 61 parts, among them IC1 XR22404, J1 USB_B_WE, J2 Conn_01x01, J3 Conn_01x01, J4 Conn_01x01, J5 Conn_01x01, J6 USB_A_shielded, J7 USB_A_shielded, J8 USB_A_shielded, J9 USB_A_shielded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

Commit message: Add files via upload
Connections:
- net USB_D_1+: now also J1.3 (D+), U1.3; no longer J1.2 (D-), U1.6
- net USB_D_1-: now also J1.2 (D-), U1.1; no longer J1.3 (D+), U1.4
- net USB_D_2+: now also FL1.1, U1.4; no longer FL1.4, U1.1
- net USB_D_2-: now also FL1.4, U1.6; no longer FL1.1, U1.3
- net USB_D_3+: now also FL1.2; no longer FL1.3
- net USB_D_3-: now also FL1.3; no longer FL1.2
Changed lines of the file:
@@
 $EndComp
 Wire Wire Line
-	1850 4300 2200 4300
+	1850 4300 2000 4300
+Wire Wire Line
+	2000 4300 2200 4300
 Wire Wire Line
 	2000 4500 2000 4300
@@
 	2000 4800 2000 5050
 Wire Wire Line
-	2000 5050 2500 5050
+	2000 5050 2400 5050
+Wire Wire Line
+	2400 5050 2500 5050
 Wire Wire Line
 	2400 5050 2400 4600
 Connection ~ 2400 5050
 Wire Wire Line
-	2600 4300 3100 4300
-Wire Wire Line
-	2950 3950 2950 4500
-Wire Wire Line
-	2750 3950 3300 3950
+	2600 4300 2950 4300
+Wire Wire Line
+	2950 4300 3100 4300
+Wire Wire Line
+	2950 3950 2950 4300
+Wire Wire Line
+	2950 4300 2950 4500
+Wire Wire Line
+	2750 3950 2950 3950
+Wire Wire Line
+	2950 3950 3300 3950
 Connection ~ 2950 3950
 Wire Wire Line
-	2800 5050 4100 5050
-Wire Wire Line
-	2950 4800 2950 5150
+	2800 5050 2950 5050
+Wire Wire Line
+	2950 5050 3550 5050
+Wire Wire Line
+	3550 5050 4100 5050
+Wire Wire Line
+	2950 4800 2950 5050
+Wire Wire Line
+	2950 5050 2950 5150
 Connection ~ 2950 4300
 Wire Wire Line
-	3400 4300 4300 4300
+	3400 4300 3550 4300
+Wire Wire Line
+	3550 4300 4100 4300
+Wire Wire Line
+	4100 4300 4300 4300
 Wire Wire Line
 	3550 4300 3550 4500
@@
 	2300 5650 2200 5650
 Wire Wire Line
-	2200 5650 2200 5950
+	2200 5650 2200 5800
+Wire Wire Line
+	2200 5800 2200 5950
 Wire Wire Line
 	2200 5800 2100 5800
@@
 	2300 6250 2200 6250
 Wire Wire Line
-	2200 6250 2200 6550
+	2200 6250 2200 6400
+Wire Wire Line
+	2200 6400 2200 6550
 Wire Wire Line
 	2200 6400 2100 6400
@@
 	2600 5650 2950 5650
 Wire Wire Line
-	2950 5650 2950 5950
+	2950 5650 2950 5800
+Wire Wire Line
+	2950 5800 2950 5950
 Wire Wire Line
 	2950 5950 2600 5950
@@
 	2600 6250 2950 6250
 Wire Wire Line
-	2950 6250 2950 6550
+	2950 6250 2950 6400
+Wire Wire Line
+	2950 6400 2950 6550
 Wire Wire Line
 	2950 6550 2600 6550
@@
 	2950 5800 3100 5800
 Wire Wire Line
-	3100 5800 3100 6700
+	3100 5800 3100 6400
+Wire Wire Line
+	3100 6400 3100 6700
 Wire Wire Line
 	3100 6400 2950 6400
@@
 Connection ~ 2950 5800
 Wire Wire Line
-	3100 6700 1700 6700
+	3100 6700 2350 6700
+Wire Wire Line
+	2350 6700 1700 6700
 Connection ~ 3100 6400
 Wire Wire Line
@@
 VCC33
 Wire Wire Line
-	6350 6250 7350 6250
+	6350 6250 6450 6250
+Wire Wire Line
+	6450 6250 7350 6250
 $Comp
 L Test_Point TP4
@@
 $EndComp
 Wire Wire Line
-	6450 6050 6450 6400
+	6450 6050 6450 6250
+Wire Wire Line
+	6450 6250 6450 6400
 Connection ~ 6450 6250
 $Comp
@@
 $EndComp
 Wire Wire Line
-	6850 6400 7350 6400
+	6850 6400 6900 6400
+Wire Wire Line
+	6900 6400 7350 6400
 Wire Wire Line
 	6450 6400 6550 6400
@@
 $Bitmap
 Pos 15800 10300
-Scale 0,750000
+Scale 0,000000
 Data
 89 50 4E 47 0D 0A 1A 0A 00 00 00 0D 49 48 44 52 00 00 00 96 00 00 00 9D 08 06 00 00 00 56 C6 81
@@
 	4200 5950 4300 5950
 Wire Wire Line
-	3600 5950 3900 5950
+	3600 5950 3750 5950
+Wire Wire Line
+	3750 5950 3900 5950
 Wire Wire Line
 	3750 5800 3750 5950
@@
 $EndComp
 Wire Wire Line
-	3600 6300 4150 6300
+	3600 6300 3850 6300
+Wire Wire Line
+	3850 6300 4150 6300
 Wire Wire Line
 	4150 6300 4150 6400
@@
 Connection ~ 3850 6300
 Wire Wire Line
-	3850 6800 4150 6800
+	3850 6800 4000 6800
+Wire Wire Line
+	4000 6800 4150 6800
 Wire Wire Line
 	4000 6900 4000 6800
@@
 L WE-TVS_Diode U1
 U 1 1 59EECDB6
-P 3250 2900
-F 0 "U1" V 2663 2950 60  0000 C CNN
-F 1 "WE-TVS_Diode" V 2769 2950 60  0000 C CNN
-F 2 "user_housing:SOT23-6L" H 3250 2900 60  0001 C CNN
-F 3 "" H 3250 2900 60  0001 C CNN
-	1    3250 2900
-	0    -1   1    0
+P 3150 2900
+F 0 "U1" V 2563 2950 60  0000 C CNN
+F 1 "WE-TVS_Diode" V 2669 2950 60  0000 C CNN
+F 2 "user_housing:SOT23-6L" H 3150 2900 60  0001 C CNN
+F 3 "" H 3150 2900 60  0001 C CNN
+	1    3150 2900
+	0    1    1    0
 $EndComp
 $Comp
@@
 	14000 2700 14000 2150
 Wire Wire Line
-	14000 2150 13500 2150
+	14000 2150 13600 2150
+Wire Wire Line
+	13600 2150 13500 2150
 Wire Wire Line
 	13600 2250 13600 2150
 Connection ~ 13600 2150
 Wire Wire Line
-	12700 2150 13200 2150
+	12700 2150 13100 2150
+Wire Wire Line
+	13100 2150 13200 2150
 Wire Wire Line
 	13100 2150 13100 2250
 Wire Wire Line
-	12700 1950 12700 2700
+	12700 1950 12700 2150
+Wire Wire Line
+	12700 2150 12700 2700
 Wire Wire Line
 	12700 2700 12400 2700
@@
 	14000 4450 14000 3900
 Wire Wire Line
-	14000 3900 13500 3900
+	14000 3900 13600 3900
+Wire Wire Line
+	13600 3900 13500 3900
 Wire Wire Line
 	13600 4000 13600 3900
 Connection ~ 13600 3900
 Wire Wire Line
-	12700 3900 13200 3900
+	12700 3900 13100 3900
+Wire Wire Line
+	13100 3900 13200 3900
 Wire Wire Line
 	13100 3900 13100 4000
 Wire Wire Line
-	12700 3700 12700 4450
+	12700 3700 12700 3900
+Wire Wire Line
+	12700 3900 12700 4450
 Wire Wire Line
 	12700 4450 12400 4450
@@
 	14000 6150 14000 5600
 Wire Wire Line
-	14000 5600 13500 5600
+	14000 5600 13600 5600
+Wire Wire Line
+	13600 5600 13500 5600
 Wire Wire Line
 	13600 5700 13600 5600
 Connection ~ 13600 5600
 Wire Wire Line
-	12700 5600 13200 5600
+	12700 5600 13100 5600
+Wire Wire Line
+	13100 5600 13200 5600
 Wire Wire Line
 	13100 5600 13100 5700
 Wire Wire Line
-	12700 5400 12700 6150
+	12700 5400 12700 5600
+Wire Wire Line
+	12700 5600 12700 6150
 Wire Wire Line
 	12700 6150 12400 6150
@@
 	14000 7850 14000 7300
 Wire Wire Line
-	14000 7300 13500 7300
+	14000 7300 13600 7300
+Wire Wire Line
+	13600 7300 13500 7300
 Wire Wire Line
 	13600 7400 13600 7300
 Connection ~ 13600 7300
 Wire Wire Line
-	12700 7300 13200 7300
+	12700 7300 13100 7300
+Wire Wire Line
+	13100 7300 13200 7300
 Wire Wire Line
 	13100 7300 13100 7400
 Wire Wire Line
-	12700 7100 12700 7850
+	12700 7100 12700 7300
+Wire Wire Line
+	12700 7300 12700 7850
 Wire Wire Line
 	12700 7850 12400 7850
@@
 	2100 3200 2750 3200
 Wire Wire Line
-	2650 2900 2750 2900
+	2550 2900 2750 2900
 Text GLabel 2100 2350 2    60   Input ~ 0
 VBUS_UP_P
@@
 L GND #PWR027
 U 1 1 59F02F3C
-P 3850 2900
-F 0 "#PWR027" H 3850 2650 50  0001 C CNN
-F 1 "GND" H 3855 2727 50  0000 C CNN
-F 2 "" H 3850 2900 50  0001 C CNN
-F 3 "" H 3850 2900 50  0001 C CNN
-	1    3850 2900
-	1    0    0    -1
-$EndComp
-Wire Wire Line
-	3650 2900 3850 2900
+P 2550 2900
+F 0 "#PWR027" H 2550 2650 50  0001 C CNN
+F 1 "GND" H 2555 2727 50  0000 C CNN
+F 2 "" H 2550 2900 50  0001 C CNN
+F 3 "" H 2550 2900 50  0001 C CNN
+	1    2550 2900
+	1    0    0    -1
+$EndComp
+Wire Wire Line
+	3650 2900 3700 2900
 Text GLabel 4750 2800 2    60   Input ~ 0
+USB_D_3-
+Text GLabel 4750 3000 2    60   Input ~ 0
 USB_D_3+
-Text GLabel 4750 3000 2    60   Input ~ 0
-USB_D_3-
 Wire Wire Line
 	4700 2800 4750 2800
 Wire Wire Line
 	4700 3000 4750 3000
-Text GLabel 2650 2900 0    60   Input ~ 0
+Text GLabel 3700 2900 2    60   Input ~ 0
 VCC_5V
 Wire Wire Line
@@
 	5400 3650 1200 3650
 Text Label 2250 3200 0    39   ~ 0
+USB_D_1+
+Text Label 2250 2600 0    39   ~ 0
 USB_D_1-
-Text Label 2250 2600 0    39   ~ 0
-USB_D_1+
 Text Label 3700 2600 0    39   ~ 0
+USB_D_2-
+Text Label 3700 3200 0    39   ~ 0
 USB_D_2+
-Text Label 3700 3200 0    39   ~ 0
-USB_D_2-
 Text Notes 12200 9900 0    59   ~ 0
 Copyright Caroline Brix 2017.\nThis documentation describes Open Hardware and is licensed under the\nCERN OHL v. 1.2.\nYou may redistribute and modify this documentation under the terms of the\nCERN OHL v.1.2. (http://ohwr.org/cernohl). This documentation is distributed\nWITHOUT ANY EXPRESS OR IMPLIED WARRANTY, INCLUDING OF\nMERCHANTABILITY, SATISFACTORY QUALITY AND FITNESS FOR A\nPARTICULAR PURPOSE. Please see the CERN OHL v.1.2 for applicable\nconditions

Commit message: no message
Changed lines of the file:
@@
 LIBS:user_FM
 LIBS:user_schalter
+LIBS:user_text
 LIBS:user_transformer
-LIBS:user_text
 LIBS:USB-Hub V2.0-cache
 EELAYER 26 0
@@
 $EndComp
 Wire Wire Line
-	1850 4300 2000 4300
-Wire Wire Line
-	2000 4300 2200 4300
+	1850 4300 2200 4300
 Wire Wire Line
 	2000 4500 2000 4300
@@
 	2000 4800 2000 5050
 Wire Wire Line
-	2000 5050 2400 5050
-Wire Wire Line
-	2400 5050 2500 5050
+	2000 5050 2500 5050
 Wire Wire Line
 	2400 5050 2400 4600
 Connection ~ 2400 5050
 Wire Wire Line
-	2600 4300 2950 4300
-Wire Wire Line
-	2950 4300 3100 4300
-Wire Wire Line
-	2950 3950 2950 4300
-Wire Wire Line
-	2950 4300 2950 4500
-Wire Wire Line
-	2750 3950 2950 3950
-Wire Wire Line
-	2950 3950 3300 3950
+	2600 4300 3100 4300
+Wire Wire Line
+	2950 3950 2950 4500
+Wire Wire Line
+	2750 3950 3300 3950
 Connection ~ 2950 3950
 Wire Wire Line
-	2800 5050 2950 5050
-Wire Wire Line
-	2950 5050 3550 5050
-Wire Wire Line
-	3550 5050 4100 5050
-Wire Wire Line
-	2950 4800 2950 5050
-Wire Wire Line
-	2950 5050 2950 5150
+	2800 5050 4100 5050
+Wire Wire Line
+	2950 4800 2950 5150
 Connection ~ 2950 4300
 Wire Wire Line
-	3400 4300 3550 4300
-Wire Wire Line
-	3550 4300 4100 4300
-Wire Wire Line
-	4100 4300 4300 4300
+	3400 4300 4300 4300
 Wire Wire Line
 	3550 4300 3550 4500
@@
 	2300 5650 2200 5650
 Wire Wire Line
-	2200 5650 2200 5800
-Wire Wire Line
-	2200 5800 2200 5950
+	2200 5650 2200 5950
 Wire Wire Line
 	2200 5800 2100 5800
@@
 	2300 6250 2200 6250
 Wire Wire Line
-	2200 6250 2200 6400
-Wire Wire Line
-	2200 6400 2200 6550
+	2200 6250 2200 6550
 Wire Wire Line
 	2200 6400 2100 6400
@@
 	2600 5650 2950 5650
 Wire Wire Line
-	2950 5650 2950 5800
-Wire Wire Line
-	2950 5800 2950 5950
+	2950 5650 2950 5950
 Wire Wire Line
 	2950 5950 2600 5950
@@
 	2600 6250 2950 6250
 Wire Wire Line
-	2950 6250 2950 6400
-Wire Wire Line
-	2950 6400 2950 6550
+	2950 6250 2950 6550
 Wire Wire Line
 	2950 6550 2600 6550
@@
 	2950 5800 3100 5800
 Wire Wire Line
-	3100 5800 3100 6400
-Wire Wire Line
-	3100 6400 3100 6700
+	3100 5800 3100 6700
 Wire Wire Line
 	3100 6400 2950 6400
@@
 Connection ~ 2950 5800
 Wire Wire Line
-	3100 6700 2350 6700
-Wire Wire Line
-	2350 6700 1700 6700
+	3100 6700 1700 6700
 Connection ~ 3100 6400
 Wire Wire Line
@@
 VCC33
 Wire Wire Line
-	6350 6250 6450 6250
-Wire Wire Line
-	6450 6250 7350 6250
+	6350 6250 7350 6250
 $Comp
 L Test_Point TP4
@@
 $EndComp
 Wire Wire Line
-	6450 6050 6450 6250
-Wire Wire Line
-	6450 6250 6450 6400
+	6450 6050 6450 6400
 Connection ~ 6450 6250
 $Comp
@@
 $EndComp
 Wire Wire Line
-	6850 6400 6900 6400
-Wire Wire Line
-	6900 6400 7350 6400
+	6850 6400 7350 6400
 Wire Wire Line
 	6450 6400 6550 6400
@@
 	4200 5950 4300 5950
 Wire Wire Line
-	3600 5950 3750 5950
-Wire Wire Line
-	3750 5950 3900 5950
+	3600 5950 3900 5950
 Wire Wire Line
 	3750 5800 3750 5950
@@
 $EndComp
 Wire Wire Line
-	3600 6300 3850 6300
-Wire Wire Line
-	3850 6300 4150 6300
+	3600 6300 4150 6300
 Wire Wire Line
 	4150 6300 4150 6400
@@
 Connection ~ 3850 6300
 Wire Wire Line
-	3850 6800 4000 6800
-Wire Wire Line
-	4000 6800 4150 6800
+	3850 6800 4150 6800
 Wire Wire Line
 	4000 6900 4000 6800
@@
 	14000 2700 14000 2150
 Wire Wire Line
-	14000 2150 13600 2150
-Wire Wire Line
-	13600 2150 13500 2150
+	14000 2150 13500 2150
 Wire Wire Line
 	13600 2250 13600 2150
 Connection ~ 13600 2150
 Wire Wire Line
-	12700 2150 13100 2150
-Wire Wire Line
-	13100 2150 13200 2150
+	12700 2150 13200 2150
 Wire Wire Line
 	13100 2150 13100 2250
 Wire Wire Line
-	12700 1950 12700 2150
-Wire Wire Line
-	12700 2150 12700 2700
+	12700 1950 12700 2700
 Wire Wire Line
 	12700 2700 12400 2700
@@
 	14000 4450 14000 3900
 Wire Wire Line
-	14000 3900 13600 3900
-Wire Wire Line
-	13600 3900 13500 3900
+	14000 3900 13500 3900
 Wire Wire Line
 	13600 4000 13600 3900
 Connection ~ 13600 3900
 Wire Wire Line
-	12700 3900 13100 3900
-Wire Wire Line
-	13100 3900 13200 3900
+	12700 3900 13200 3900
 Wire Wire Line
 	13100 3900 13100 4000
 Wire Wire Line
-	12700 3700 12700 3900
-Wire Wire Line
-	12700 3900 12700 4450
+	12700 3700 12700 4450
 Wire Wire Line
 	12700 4450 12400 4450
@@
 	14000 6150 14000 5600
 Wire Wire Line
-	14000 5600 13600 5600
-Wire Wire Line
-	13600 5600 13500 5600
+	14000 5600 13500 5600
 Wire Wire Line
 	13600 5700 13600 5600
 Connection ~ 13600 5600
 Wire Wire Line
-	12700 5600 13100 5600
-Wire Wire Line
-	13100 5600 13200 5600
+	12700 5600 13200 5600
 Wire Wire Line
 	13100 5600 13100 5700
 Wire Wire Line
-	12700 5400 12700 5600
-Wire Wire Line
-	12700 5600 12700 6150
+	12700 5400 12700 6150
 Wire Wire Line
 	12700 6150 12400 6150
@@
 	14000 7850 14000 7300
 Wire Wire Line
-	14000 7300 13600 7300
-Wire Wire Line
-	13600 7300 13500 7300
+	14000 7300 13500 7300
 Wire Wire Line
 	13600 7400 13600 7300
 Connection ~ 13600 7300
 Wire Wire Line
-	12700 7300 13100 7300
-Wire Wire Line
-	13100 7300 13200 7300
+	12700 7300 13200 7300
 Wire Wire Line
 	13100 7300 13100 7400
 Wire Wire Line
-	12700 7100 12700 7300
-Wire Wire Line
-	12700 7300 12700 7850
+	12700 7100 12700 7850
 Wire Wire Line
 	12700 7850 12400 7850

Commit message: no message
Parts:
- added Txt2: OSHW, Symbols:OSHW-Logo2_7.3x6mm_SilkScreen, symbol OSHW
Connections:
- net DM1_1+: now also FL5.4; no longer FL5.1
- net DM1_1-: now also FL5.1; no longer FL5.4
- net DM1_2+: now also FL5.3, U5.1; no longer FL5.2, U5.3
- net DM1_2-: now also FL5.2, U5.3; no longer FL5.3, U5.1
- net DM1_3+: now also U5.6; no longer U5.4
- net DM1_3-: now also U5.4; no longer U5.6
- net DM2_1+: now also FL4.4; no longer FL4.1
- net DM2_1-: now also FL4.1; no longer FL4.4
- net DM2_2+: now also FL4.3, U4.1; no longer FL4.2, U4.3
- net DM2_2-: now also FL4.2, U4.3; no longer FL4.3, U4.1
- net DM2_3+: now also U4.6; no longer U4.4
- net DM2_3-: now also U4.4; no longer U4.6
- net DM3_1+: now also FL3.4; no longer FL3.1
- net DM3_1-: now also FL3.1; no longer FL3.4
- net DM3_2+: now also FL3.3, U3.1; no longer FL3.2, U3.3
- net DM3_2-: now also FL3.2, U3.3; no longer FL3.3, U3.1
- net DM3_3+: now also U3.6; no longer U3.4
- net DM3_3-: now also U3.4; no longer U3.6
- net DM4_1+: now also FL2.4; no longer FL2.1
- net DM4_1-: now also FL2.1; no longer FL2.4
- net DM4_2+: now also FL2.3, U2.1; no longer FL2.2, U2.3
- net DM4_2-: now also FL2.2, U2.3; no longer FL2.3, U2.1
- net DM4_3+: now also U2.6; no longer U2.4
- net DM4_3-: now also U2.4; no longer U2.6
Other:
- moved on the sheet: U2, U3, U4, U5
Changed lines of the file:
@@
 F 3 "" V 10700 2740 50  0000 C CNN
 	1    10700 2700
-	1    0    0    -1
+	1    0    0    1
 $EndComp
 $Comp
@@
 F 3 "" H 11900 2700 60  0001 C CNN
 	1    11900 2700
-	0    1    1    0
+	0    1    -1   0
 $EndComp
 $Comp
@@
 F 3 "" V 10700 4490 50  0000 C CNN
 	1    10700 4450
-	1    0    0    -1
+	1    0    0    1
 $EndComp
 $Comp
@@
 F 3 "" H 11900 4450 60  0001 C CNN
 	1    11900 4450
-	0    1    1    0
+	0    1    -1   0
 $EndComp
 $Comp
@@
 F 3 "" V 10700 6190 50  0000 C CNN
 	1    10700 6150
-	1    0    0    -1
+	1    0    0    1
 $EndComp
 $Comp
@@
 F 3 "" H 11900 6150 60  0001 C CNN
 	1    11900 6150
-	0    1    1    0
+	0    1    -1   0
 $EndComp
 $Comp
@@
 F 3 "" V 10700 7890 50  0000 C CNN
 	1    10700 7850
-	1    0    0    -1
+	1    0    0    1
 $EndComp
 $Comp
@@
 F 3 "" H 11900 7850 60  0001 C CNN
 	1    11900 7850
-	0    1    1    0
+	0    1    -1   0
 $EndComp
 $Comp
@@
 	1    0    0    -1
 $EndComp
+$Comp
+L OSHW Txt2
+U 1 1 59F261AA
+P 10600 10900
+F 0 "Txt2" H 10625 10953 60  0000 L CNN
+F 1 "OSHW" H 10625 10847 60  0000 L CNN
+F 2 "Symbols:OSHW-Logo2_7.3x6mm_SilkScreen" H 10600 10900 60  0001 C CNN
+F 3 "" H 10600 10900 60  0001 C CNN
+	1    10600 10900
+	1    0    0    -1
+$EndComp
